Commit message: Nav2 + AMCL per robot, complete factory world with running lines
- navigation.launch.py: one map_server for the fleet, per robot a component
  container with AMCL, controller_server (Regulated Pure Pursuit, local
  costmap from 2D lidar + RGB-D points) and collision_monitor; optional
  planner/behavior/bt_navigator (nav2_full_stack:=true)
- robot_agent driver:=nav2 sends the lane route granted by traffic control
  to FollowPath, lane speed limits on speed_limit, pose = AMCL estimate
  composed with wheel odometry; progress tracking tolerates corner cutting;
  local costmap recovery after controller failures
- Gazebo: wheel odometry for AMCL (ground truth kept on /<id>/ground_truth),
  cargo lift joint shows goods on board, bridge for line state and lifts
- LineAnimator gz-sim system: products move on all 8 conveyors and stop
  when the MES reports a line starved / blocked
- world generator: walls, windows, roller doors, columns, roof lights,
  racks with goods, 4 production + 4 packaging lines, office, trucks;
  opaque static geometry baked into one OBJ (one sub-mesh per material)
  so the fleet's sensors render fast; AMCL map sliced at the lidar plane
- dashboard / RViz: new layout labels, task-priority explanation, AMCL
  particles, collision monitor zones and local costmap
- README rewritten for the new factory, Nav2 and task-based priority

Co-Authored-By: Claude Opus 5.5 <noreply@anthropic.com>
Claude-Session: https://claude.ai/code/session_01AjxY7Qcftyxs4iYRzGLXQF

File: src/amr_description/urdf/amr.gazebo.xacro (robot description, xacro)
@@ -4,5 +4,6 @@
      can serve the whole fleet. -->
 <robot xmlns:xacro="http://www.ros.org/wiki/xacro">
-  <xacro:macro name="amr_gazebo" params="ns wheel_sep wheel_r camera camera_rate lidar_rate">
+  <xacro:macro name="amr_gazebo" params="ns wheel_sep wheel_r camera camera_rate lidar_rate odom:=ground_truth">
+    <xacro:property name="wheel_odom" value="${odom == 'wheel'}"/>
     <gazebo>
       <!-- 2 driven wheels -->
@@ -21,17 +22,30 @@
         <min_angular_acceleration>-3.5</min_angular_acceleration>
         <topic>/${ns}/cmd_vel</topic>
-        <odom_topic>/${ns}/wheel_odom</odom_topic>
-        <tf_topic>/${ns}/wheel_tf</tf_topic>
+        <xacro:if value="${wheel_odom}">
+          <!-- wheel odometry: drifts like on a real AMR, AMCL publishes map->odom -->
+          <odom_topic>/${ns}/odom</odom_topic>
+          <tf_topic>/${ns}/tf</tf_topic>
+        </xacro:if>
+        <xacro:unless value="${wheel_odom}">
+          <odom_topic>/${ns}/wheel_odom</odom_topic>
+          <tf_topic>/${ns}/wheel_tf</tf_topic>
+        </xacro:unless>
         <frame_id>${ns}/odom</frame_id>
         <child_frame_id>${ns}/base_footprint</child_frame_id>
-        <odom_publish_frequency>20</odom_publish_frequency>
+        <odom_publish_frequency>30</odom_publish_frequency>
       </plugin>
-      <!-- map-aligned odometry + TF (stands in for an on-board localisation) -->
+      <!-- exact pose: odometry in ground-truth mode, /<ns>/ground_truth otherwise -->
       <plugin filename="gz-sim-odometry-publisher-system" name="gz::sim::systems::OdometryPublisher">
         <odom_frame>${ns}/odom</odom_frame>
         <robot_base_frame>${ns}/base_footprint</robot_base_frame>
         <odom_publish_frequency>30</odom_publish_frequency>
-        <odom_topic>/${ns}/odom</odom_topic>
-        <tf_topic>/${ns}/tf</tf_topic>
+        <xacro:if value="${wheel_odom}">
+          <odom_topic>/${ns}/ground_truth</odom_topic>
+          <tf_topic>/${ns}/ground_truth_tf</tf_topic>
+        </xacro:if>
+        <xacro:unless value="${wheel_odom}">
+          <odom_topic>/${ns}/odom</odom_topic>
+          <tf_topic>/${ns}/tf</tf_topic>
+        </xacro:unless>
         <dimensions>2</dimensions>
       </plugin>
@@ -40,4 +54,19 @@
         <joint_name>left_wheel_joint</joint_name>
         <joint_name>right_wheel_joint</joint_name>
+        <joint_name>cargo_joint</joint_name>
+      </plugin>
+      <!-- cargo lift: 0 = hidden in the chassis, 0.235 = load on the deck.
+           Force PID (velocity commands do not move a prismatic joint in gz-sim 8). -->
+      <plugin filename="gz-sim-joint-position-controller-system"
+              name="gz::sim::systems::JointPositionController">
+        <joint_name>cargo_joint</joint_name>
+        <topic>/${ns}/cargo_lift</topic>
+        <p_gain>400</p_gain>
+        <i_gain>40</i_gain>
+        <d_gain>40</d_gain>
+        <i_max>50</i_max>
+        <i_min>-50</i_min>
+        <cmd_max>150</cmd_max>
+        <cmd_min>-150</cmd_min>
       </plugin>
     </gazebo>

File: src/amr_description/urdf/amr.urdf.xacro (robot description, xacro)
@@ -19,4 +19,5 @@
   <xacro:arg name="camera_rate" default="5"/>
   <xacro:arg name="lidar_rate" default="10"/>
+  <xacro:arg name="odom" default="ground_truth"/>   <!-- ground_truth | wheel (for AMCL / Nav2) -->
   <xacro:property name="ns" value="$(arg robot_name)"/>
   <xacro:property name="pfx" value=""/>  <!-- frames are prefixed by robot_state_publisher (frame_prefix) -->
@@ -208,9 +209,35 @@
     <origin rpy="${-PI/2} 0 ${-PI/2}"/>
   </joint>
+  <!-- ============================================== cargo (visual load) -->
+  <!-- Lifted onto the deck while the AMR carries goods, hidden inside the
+       chassis otherwise (prismatic joint driven by a position controller). -->
+  <material name="cargo"><color rgba="0.74 0.56 0.34 1"/></material>
+  <link name="${pfx}cargo_link">
+    <visual>
+      <geometry><box size="0.56 0.40 0.22"/></geometry>
+      <material name="cargo"/>
+    </visual>
+    <visual>
+      <origin xyz="0 0 0.111"/>
+      <geometry><box size="0.57 0.06 0.004"/></geometry>
+      <material name="deck"/>
+    </visual>
+    <inertial>
+      <mass value="1.0"/>
+      <inertia ixx="0.02" ixy="0" ixz="0" iyy="0.03" iyz="0" izz="0.04"/>
+    </inertial>
+  </link>
+  <joint name="cargo_joint" type="prismatic">
+    <parent link="${pfx}base_link"/>
+    <child link="${pfx}cargo_link"/>
+    <origin xyz="0 0 ${0.17 - wheel_r}"/>
+    <axis xyz="0 0 1"/>
+    <limit lower="0.0" upper="0.24" effort="300" velocity="0.5"/>
+  </joint>
   <xacro:if value="$(arg gazebo)">
     <xacro:include filename="$(find amr_description)/urdf/amr.gazebo.xacro"/>
     <xacro:amr_gazebo ns="${ns}" wheel_sep="${wheel_sep}" wheel_r="${wheel_r}"
                       camera="$(arg camera)" camera_rate="$(arg camera_rate)"
-                      lidar_rate="$(arg lidar_rate)"/>
+                      lidar_rate="$(arg lidar_rate)" odom="$(arg odom)"/>
   </xacro:if>
 </robot>

Commit message: One 270 deg front lidar with a scanner slot in the chassis
- gpu_lidar -135..+135 deg, 541 samples (0.5 deg), still one sensor at the
  front centre, 0.20 m high
- the chassis is built in three layers; the middle one (0.17-0.23 m) is cut
  back to x = 0.18 so the +-135 deg rays pass along the sides of the body
- the unloaded cargo box is lowered below the floor (-0.30) instead of
  resting inside the chassis, where it crossed the lidar plane (found by
  removing visuals one by one: 34 self hits at 0.2 m -> 0)
- kinematic simulator: 270 deg scans, 1 deg resolution

Co-Authored-By: Claude Opus 5.5 <noreply@anthropic.com>
Claude-Session: https://claude.ai/code/session_01AjxY7Qcftyxs4iYRzGLXQF

File: src/amr_description/urdf/amr.gazebo.xacro (robot description, xacro)
@@ -56,5 +56,5 @@
         <joint_name>cargo_joint</joint_name>
       </plugin>
-      <!-- cargo lift: 0 = hidden in the chassis, 0.235 = load on the deck.
+      <!-- cargo lift: -0.30 = no load (below the floor), 0.235 = load on the deck.
            Force PID (velocity commands do not move a prismatic joint in gz-sim 8). -->
       <plugin filename="gz-sim-joint-position-controller-system"
@@ -62,4 +62,5 @@
         <joint_name>cargo_joint</joint_name>
         <topic>/${ns}/cargo_lift</topic>
+        <initial_position>-0.30</initial_position>
         <p_gain>400</p_gain>
         <i_gain>40</i_gain>
@@ -71,5 +72,5 @@
       </plugin>
     </gazebo>
-    <!-- 2D lidar: 180 deg in front of the robot -->
+    <!-- 2D lidar: 270 deg (+-135 deg) at the front of the robot, 0.5 deg resolution -->
     <gazebo reference="lidar_link">
       <sensor name="lidar" type="gpu_lidar">
@@ -82,8 +83,8 @@
           <scan>
             <horizontal>
-              <samples>361</samples>
+              <samples>541</samples>
               <resolution>1</resolution>
-              <min_angle>-1.5708</min_angle>
-              <max_angle>1.5708</max_angle>
+              <min_angle>-2.35619</min_angle>
+              <max_angle>2.35619</max_angle>
             </horizontal>
             <vertical>

File: src/amr_description/urdf/amr.urdf.xacro (robot description, xacro)
@@ -2,6 +2,6 @@
 <!--
   Factory AMR: differential drive with 2 driven wheels (centre of the chassis)
-  and 4 free (caster) wheels at the corners, one 2D lidar at the front and one
-  RGB-D (3D) camera.  Footprint 0.80 m x 0.56 m, payload deck at 0.29 m.
+  and 4 free (caster) wheels at the corners, one 270 deg 2D lidar at the front
+  and one RGB-D (3D) camera.  Footprint 0.80 m x 0.56 m, payload deck at 0.29 m.
   xacro args
     robot_name   namespace / frame prefix, e.g. amr_01   (frames: amr_01/base_link ...)
@@ -35,4 +35,8 @@
   <xacro:property name="caster_y" value="0.17"/>
   <xacro:property name="mass_body" value="45.0"/>
+  <!-- scanner slot: height band around the lidar plane (0.20 m) and how far it is cut back -->
+  <xacro:property name="slot_z0" value="0.17"/>
+  <xacro:property name="slot_z1" value="0.23"/>
+  <xacro:property name="slot_x" value="0.18"/>
   <material name="body"><color rgba="$(arg color)"/></material>
   <material name="deck"><color rgba="0.20 0.21 0.23 1"/></material>
@@ -50,7 +54,25 @@
   <link name="${pfx}base_footprint"/>
   <link name="${pfx}base_link">
-    <visual>
-      <origin xyz="0 0 ${clearance + body_h/2 - wheel_r}"/>
-      <geometry><box size="${body_l} ${body_w} ${body_h}"/></geometry>
+    <!-- chassis in three layers: the middle layer (lidar plane +-3 cm) is cut back
+         to x = 0.18 so the 270 deg front scanner sees past the body up to +-135 deg
+         (like the scanner slot of a real AMR) -->
+    <visual>
+      <origin xyz="0 0 ${(clearance + slot_z0) / 2 - wheel_r}"/>
+      <geometry><box size="${body_l} ${body_w} ${slot_z0 - clearance}"/></geometry>
+      <material name="body"/>
+    </visual>
+    <visual>
+      <origin xyz="${(slot_x - body_l/2) / 2} 0 ${(slot_z0 + slot_z1) / 2 - wheel_r}"/>
+      <geometry><box size="${slot_x + body_l/2} ${body_w} ${slot_z1 - slot_z0}"/></geometry>
+      <material name="body"/>
+    </visual>
+    <visual>
+      <origin xyz="${slot_x + 0.003} 0 ${(slot_z0 + slot_z1) / 2 - wheel_r}"/>
+      <geometry><box size="0.006 ${body_w - 0.02} ${slot_z1 - slot_z0 - 0.01}"/></geometry>
+      <material name="sensor"/>
+    </visual>
+    <visual>
+      <origin xyz="0 0 ${(slot_z1 + clearance + body_h) / 2 - wheel_r}"/>
+      <geometry><box size="${body_l} ${body_w} ${clearance + body_h - slot_z1}"/></geometry>
       <material name="body"/>
     </visual>
@@ -184,5 +206,6 @@
     <parent link="${pfx}base_link"/>
     <child link="${pfx}lidar_link"/>
-    <!-- front centre, 0.20 m above the floor, in front of the bumper -->
+    <!-- front centre, 0.20 m above the floor, in front of the bumper; 270 deg field
+         of view through the scanner slot of the chassis -->
     <origin xyz="0.43 0 ${0.20 - wheel_r}"/>
   </joint>
@@ -210,6 +233,7 @@
   </joint>
   <!-- ============================================== cargo (visual load) -->
-  <!-- Lifted onto the deck while the AMR carries goods, hidden inside the
-       chassis otherwise (prismatic joint driven by a position controller). -->
+  <!-- Lifted onto the deck (0.235) while the AMR carries goods, lowered below the
+       floor (-0.30) otherwise: kept inside the chassis it would cross the lidar plane
+       in the scanner slot (prismatic joint driven by a position controller). -->
   <material name="cargo"><color rgba="0.74 0.56 0.34 1"/></material>
   <link name="${pfx}cargo_link">
@@ -233,5 +257,5 @@
     <origin xyz="0 0 ${0.17 - wheel_r}"/>
     <axis xyz="0 0 1"/>
-    <limit lower="0.0" upper="0.24" effort="300" velocity="0.5"/>
+    <limit lower="-0.30" upper="0.24" effort="300" velocity="1.0"/>
   </joint>
   <xacro:if value="$(arg gazebo)">

Commit message: Staggered charging, walkway crossings, camera load, dock fix, docs
- Opportunistic charging only while the fleet has spare robots, at most 40%
  of it away at once (5 robots +7% finished goods, max away 4 -> 2 with 7)
- Edges crossing a workers' walkway limited to 0.9 m/s
- RGB-D 160x120 for robots whose images are not shown (4x smaller clouds)
- Collision monitor stop zone back to 0.75 m: at 0.85 m it saw the charger
  contact arm at the dock staging pose and froze undocked robots
- Quiet Ctrl+C on Humble (context shut down while spinning)
- README: smoothness tooling, measured results, fleet sizing

Co-Authored-By: Claude Opus 5.5 <noreply@anthropic.com>
Claude-Session: https://claude.ai/code/session_01D1ezER7WBS8PaJLbYYgdBA

File: src/amr_description/urdf/amr.gazebo.xacro (robot description, xacro)
@@ -4,5 +4,5 @@
      can serve the whole fleet. -->
 <robot xmlns:xacro="http://www.ros.org/wiki/xacro">
-  <xacro:macro name="amr_gazebo" params="ns wheel_sep wheel_r camera camera_rate lidar_rate odom:=ground_truth">
+  <xacro:macro name="amr_gazebo" params="ns wheel_sep wheel_r camera camera_rate lidar_rate odom:=ground_truth camera_width:=320 camera_height:=240">
     <xacro:property name="wheel_odom" value="${odom == 'wheel'}"/>
     <gazebo>
@@ -120,6 +120,6 @@
             <horizontal_fov>1.50</horizontal_fov>
             <image>
-              <width>320</width>
-              <height>240</height>
+              <width>${camera_width}</width>
+              <height>${camera_height}</height>
               <format>R8G8B8</format>
             </image>

File: src/amr_description/urdf/amr.urdf.xacro (robot description, xacro)
@@ -18,4 +18,6 @@
   <xacro:arg name="camera" default="true"/>
   <xacro:arg name="camera_rate" default="5"/>
+  <xacro:arg name="camera_width" default="320"/>    <!-- RGB-D resolution (point cloud size) -->
+  <xacro:arg name="camera_height" default="240"/>
   <xacro:arg name="lidar_rate" default="10"/>
   <xacro:arg name="odom" default="ground_truth"/>   <!-- ground_truth | wheel (for AMCL / Nav2) -->
@@ -263,4 +265,5 @@
     <xacro:amr_gazebo ns="${ns}" wheel_sep="${wheel_sep}" wheel_r="${wheel_r}"
                       camera="$(arg camera)" camera_rate="$(arg camera_rate)"
+                      camera_width="$(arg camera_width)" camera_height="$(arg camera_height)"
                       lidar_rate="$(arg lidar_rate)" odom="$(arg odom)"/>
   </xacro:if>
